Commit message: Remove unused initial test scripts

File: assets/generated/ssk_iiwa7_gpu_heart.urdf (robot description, URDF)
Before this commit: robot iiwa7, 12 links, 11 joints
Links:
- link visual_sculpting_tool: geometry collision cylinder length=0.07 radius=0.015; visual cylinder length=0.07 radius=0.015
Joints:
- joint visual_sculpting_tip_joint: origin xyz=0 0 0.08 rpy=0 0 0 -> xyz=0 0 0.07 rpy=0 0 0

File: assets/generated/ssk_iiwa7_visual_sculpting.urdf (robot description, URDF)
Before this commit: robot iiwa7, 12 links, 11 joints
Links:
- link visual_sculpting_tip: mass None -> 0.02; geometry collision sphere radius=0.015; visual sphere radius=0.015
- link visual_sculpting_tool: mass 0.03 -> 0.08; geometry collision cylinder length=0.06 radius=0.014; visual cylinder length=0.06 radius=0.014
Joints:
- joint visual_sculpting_tip_joint: origin xyz=0 0 0.025 rpy=0 0 0 -> xyz=0 0 0.075 rpy=0 0 0
- joint visual_sculpting_tool_joint: origin xyz=0 0 0.002 rpy=0 0 0 -> xyz=0 0 0.0015 rpy=0 0 0
